Commit message: added turret and joint for camera.

File: src/description/urdf/robot_base.xacro (robot description, xacro)
@@ -92,12 +92,30 @@
     <origin xyz="0.11 0 0.15"/>
   </joint>
-  <link name="camera_link">
-    <origin xyz="0.15 0 0.12" rpy="0 0 0"/>
-  </link>
-  <joint name="camera_joint" type="fixed">
-    <parent link="base_link"/>
-    <child link="camera_link"/>
-    <origin xyz="0.15 0 0.12"/>
-  </joint>
+  <!-- ================= PAN LINK ================= -->
+<link name="pan_link">
+  <visual>
+    <geometry>
+      <cylinder radius="0.05" length="0.02"/>
+    </geometry>
+    <material name="gray">
+      <color rgba="0.6 0.6 0.6 1.0"/>
+    </material>
+  </visual>
+</link>
+<joint name="pan_joint" type="continuous">
+  <parent link="base_link"/>
+  <child link="pan_link"/>
+  <origin xyz="0.15 0 0.12"/>
+  <axis xyz="0 0 1"/>
+</joint>
+<link name="camera_link"/>
+  <!-- ================= TILT JOINT ================= -->
+<joint name="tilt_joint" type="revolute">
+  <parent link="pan_link"/>
+  <child link="camera_link"/>
+  <origin xyz="0 0 0.05"/>
+  <axis xyz="0 1 0"/>
+  <limit lower="-1.57" upper="1.57" effort="1" velocity="1"/>
+</joint>
   <xacro:macro name="wheel" params="name x y">
     <link name="${name}_link">

File: src/description/urdf/robot_sensors.xacro (robot description, xacro)
@@ -1,62 +1,68 @@
 <?xml version="1.0"?>
 <robot xmlns:xacro="http://www.ros.org/wiki/xacro">
-  <xacro:macro name="sensors">
-    <gazebo reference="imu_link">
-      <sensor name="imu_sensor" type="imu">
-        <always_on>true</always_on>
-        <update_rate>100</update_rate>
-        <topic>/imu</topic>
-      </sensor>
-    </gazebo>
-    <gazebo reference="gps_link">
-      <sensor name="gps_sensor" type="navsat">
-        <always_on>true</always_on>
-        <update_rate>5</update_rate>
-        <topic>/gps</topic>
-      </sensor>
-    </gazebo>
-    <gazebo reference="lidar_link">
-      <sensor name="lidar_sensor" type="gpu_lidar">
-        <always_on>true</always_on>
-        <update_rate>10</update_rate>
-        <topic>/scan</topic>
-        <visualize>true</visualize>
-        <frame_id>lidar_link</frame_id>
-        <lidar>
-          <scan>
-            <horizontal>
-              <samples>360</samples>
-              <resolution>1</resolution>
-              <min_angle>-3.14159</min_angle>
-              <max_angle>3.14159</max_angle>
-            </horizontal>
-          </scan>
-          <range>
-            <min>0.1</min>
-            <max>10.0</max>
-            <resolution>0.01</resolution>
-          </range>
-        </lidar>
-      </sensor>
-    </gazebo>
-    <gazebo reference="camera_link">
-      <sensor name="camera_sensor" type="camera">
-        <always_on>true</always_on>
-        <update_rate>30</update_rate>
-        <topic>/camera/image_raw</topic>
-        <camera>
-          <horizontal_fov>1.047</horizontal_fov>
-          <image>
-            <width>640</width>
-            <height>480</height>
-            <format>R8G8B8</format>
-          </image>
-          <clip>
-            <near>0.1</near>
-            <far>100</far>
-          </clip>
-        </camera>
-      </sensor>
-    </gazebo>
-  </xacro:macro>
+<xacro:macro name="sensors">
+  <!-- ================= IMU ================= -->
+  <gazebo reference="imu_link">
+    <sensor name="imu_sensor" type="imu">
+      <always_on>true</always_on>
+      <update_rate>100</update_rate>
+      <topic>/imu</topic>
+    </sensor>
+  </gazebo>
+  <!-- ================= GPS ================= -->
+  <gazebo reference="gps_link">
+    <sensor name="gps_sensor" type="navsat">
+      <always_on>true</always_on>
+      <update_rate>5</update_rate>
+      <topic>/gps</topic>
+    </sensor>
+  </gazebo>
+  <!-- ================= LIDAR ================= -->
+  <gazebo reference="lidar_link">
+    <sensor name="lidar_sensor" type="gpu_lidar">
+      <always_on>true</always_on>
+      <update_rate>10</update_rate>
+      <topic>/scan</topic>
+      <visualize>true</visualize>
+      <frame_id>lidar_link</frame_id>
+      <lidar>
+        <scan>
+          <horizontal>
+            <samples>360</samples>
+            <resolution>1</resolution>
+            <min_angle>-3.14159</min_angle>
+            <max_angle>3.14159</max_angle>
+          </horizontal>
+        </scan>
+        <range>
+          <min>0.1</min>
+          <max>10.0</max>
+          <resolution>0.01</resolution>
+        </range>
+      </lidar>
+    </sensor>
+  </gazebo>
+  <!-- ================= CAMERA (ON TURRET) ================= -->
+  <gazebo reference="camera_link">
+    <sensor name="camera_sensor" type="camera">
+      <always_on>true</always_on>
+      <update_rate>30</update_rate>
+      <topic>/camera/image_raw</topic>
+      <!-- IMPORTANT ADD -->
+      <frame_id>camera_link</frame_id>
+      <camera>
+        <horizontal_fov>1.047</horizontal_fov>
+        <image>
+          <width>640</width>
+          <height>480</height>
+          <format>R8G8B8</format>
+        </image>
+        <clip>
+          <near>0.1</near>
+          <far>100</far>
+        </clip>
+      </camera>
+    </sensor>
+  </gazebo>
+</xacro:macro>
 </robot>

Commit message: added links justifiables for gz crash problem

File: src/description/urdf/robot_base.xacro (robot description, xacro)
@@ -102,12 +102,50 @@
     </material>
   </visual>
+  <gazebo reference="pan_link">
+  <gravity>true</gravity>
+</gazebo>
+  <collision>
+    <geometry>
+      <cylinder radius="0.05" length="0.02"/>
+    </geometry>
+  </collision>
+  <inertial>
+    <mass value="0.5"/>
+    <origin xyz="0 0 0"/>
+    <inertia
+      ixx="0.01" iyy="0.01" izz="0.01"
+      ixy="0" ixz="0" iyz="0"/>
+  </inertial>
 </link>
-<joint name="pan_joint" type="continuous">
+<joint name="pan_joint" type="revolute">
   <parent link="base_link"/>
   <child link="pan_link"/>
   <origin xyz="0.15 0 0.12"/>
   <axis xyz="0 0 1"/>
+  <limit lower="-3.14" upper="3.14" effort="10" velocity="1.0"/>
+  <dynamics damping="0.1" friction="0.1"/>
 </joint>
-<link name="camera_link"/>
+<link name="camera_link">
+  <visual>
+    <geometry>
+      <box size="0.05 0.05 0.05"/>
+    </geometry>
+    <material name="black">
+      <color rgba="0.1 0.1 0.1 1"/>
+    </material>
+  </visual>
+  <collision>
+    <geometry>
+      <box size="0.05 0.05 0.05"/>
+    </geometry>
+  </collision>
+  <inertial>
+    <mass value="0.3"/>
+    <origin xyz="0 0 0"/>
+    <inertia
+      ixx="0.005" iyy="0.005" izz="0.005"
+      ixy="0" ixz="0" iyz="0"/>
+  </inertial>
+</link>
   <!-- ================= TILT JOINT ================= -->
 <joint name="tilt_joint" type="revolute">
@@ -116,5 +154,6 @@
   <origin xyz="0 0 0.05"/>
   <axis xyz="0 1 0"/>
-  <limit lower="-1.57" upper="1.57" effort="1" velocity="1"/>
+  <limit lower="-1.57" upper="1.57" effort="10" velocity="1.0"/>
+  <dynamics damping="0.1" friction="0.1"/>
 </joint>
   <xacro:macro name="wheel" params="name x y">

File: src/description/urdf/robot_control.xacro (robot description, xacro)
@@ -26,4 +26,14 @@
       <state_interface name="velocity"/>
     </joint>
+    <joint name="pan_joint">
+  <command_interface name="position"/>
+  <state_interface name="position"/>
+  <state_interface name="velocity"/>
+</joint>
+<joint name="tilt_joint">
+  <command_interface name="position"/>
+  <state_interface name="position"/>
+  <state_interface name="velocity"/>
+</joint>
   </ros2_control>
 </xacro:macro>

Commit message: Revert "lane costmap injection started"
This reverts commit d36de82be99716132c622555bfed40b52a43b174.

File: src/description/urdf/robot_base.xacro (robot description, xacro)
@@ -92,5 +92,5 @@
       <parent link="base_link"/>
       <child link="camera_link"/>
-      <origin xyz="0.15 0 1"/>
+      <origin xyz="0.15 0 0.12"/>
     </joint>
     <xacro:macro name="wheel" params="name x y">

Commit message: Revert "more progress"
This reverts commit c822f234c4abdb127fe034871d990dfbe5951070.

File: src/description/urdf/robot_base.xacro (robot description, xacro)
@@ -92,5 +92,5 @@
       <parent link="base_link"/>
       <child link="camera_link"/>
-      <origin xyz="0.15 0 2" rpy="0 0.7 0"/>
+      <origin xyz="0.15 0 1"/>
     </joint>
     <xacro:macro name="wheel" params="name x y">

Commit message: Revert "made changes"
This reverts commit cba1a0756ca5af382cb21d8c56b6aed8f503c80f.

File: src/description/urdf/robot_base.xacro (robot description, xacro)
@@ -92,5 +92,5 @@
       <parent link="base_link"/>
       <child link="camera_link"/>
-      <origin xyz="0.15 0 2" rpy="0 0.4 0"/>
+      <origin xyz="0.15 0 2" rpy="0 0.7 0"/>
     </joint>
     <xacro:macro name="wheel" params="name x y">

Commit message: Revert "little little changes"
This reverts commit 1c10a4afae14952abd2d9e2f38727e6c8a91ddec.

File: src/description/urdf/robot_base.xacro (robot description, xacro)
@@ -1,139 +1,149 @@
 <?xml version="1.0"?>
 <robot xmlns:xacro="http://www.ros.org/wiki/xacro">
-  <xacro:macro name="base">
-    <xacro:property name="base_length" value="0.5"/>
-    <xacro:property name="base_width" value="0.4"/>
-    <xacro:property name="base_height" value="0.2"/>
-    <xacro:property name="wheel_radius" value="0.075"/>
-    <xacro:property name="wheel_width" value="0.04"/>
-    <xacro:property name="wheel_x_offset" value="0.18"/>
-    <xacro:property name="wheel_y_offset" value="0.22"/>
-    <link name="base_link">
+<xacro:macro name="base">
+  <xacro:property name="base_length" value="0.5"/>
+  <xacro:property name="base_width" value="0.4"/>
+  <xacro:property name="base_height" value="0.2"/>
+  <xacro:property name="wheel_radius" value="0.075"/>
+  <xacro:property name="wheel_width" value="0.04"/>
+  <xacro:property name="wheel_x_offset" value="0.18"/>
+  <xacro:property name="wheel_y_offset" value="0.22"/>
+<link name="base_footprint"/>
+<joint name="base_footprint_joint" type="fixed">
+  <parent link="base_footprint"/>
+  <child link="base_link"/>
+  <origin xyz="0 0 0" rpy="0 0 0"/>
+</joint>
+  <link name="base_link">
+    <visual>
+      <geometry>
+        <box size="${base_length} ${base_width} ${base_height}"/>
+      </geometry>
+      <origin xyz="0 0 ${base_height/2 + 0.05}"/>
+      <material name="body_color">
+        <color rgba="0.15 0.15 0.18 1"/>
+      </material>
+    </visual>
+    <collision>
+      <geometry>
+        <box size="${base_length} ${base_width} ${base_height}"/>
+      </geometry>
+      <origin xyz="0 0 ${base_height/2 + 0.05}"/>
+    </collision>
+    <inertial>
+      <mass value="10.0"/>
+      <origin xyz="0 0 ${base_height/2 + 0.05}"/>
+      <inertia
+        ixx="0.2"
+        iyy="0.2"
+        izz="0.2"
+        ixy="0" ixz="0" iyz="0"/>
+    </inertial>
+  </link>
+  <gazebo reference="base_link">
+    <self_collide>false</self_collide>
+  </gazebo>
+  <link name="imu_link">
+    <visual>
+      <geometry>
+        <box size="0.03 0.03 0.02"/>
+      </geometry>
+      <material name="orange">
+        <color rgba="1 0.5 0 1"/>
+      </material>
+      <origin xyz="0 0 0.15" rpy="0 0 0"/>
+    </visual>
+  </link>
+  <joint name="imu_joint" type="fixed">
+    <parent link="base_link"/>
+    <child link="imu_link"/>
+    <origin xyz="0 0 0.15"/>
+  </joint>
+  <link name="gps_link">
+    <visual>
+      <geometry>
+        <box size="0.03 0.03 0.02"/>
+      </geometry>
+      <material name="white">
+        <color rgba="1 1 1 1"/>
+      </material>
+      <origin xyz="0 0 0.2" rpy="0 0 0"/>
+    </visual>
+  </link>
+  <joint name="gps_joint" type="fixed">
+    <parent link="base_link"/>
+    <child link="gps_link"/>
+    <origin xyz="0 0 0.2"/>
+  </joint>
+  <link name="lidar_link">
+    <visual>
+      <geometry>
+        <cylinder radius="0.04" length="0.05"/>
+      </geometry>
+      <origin xyz="0.1 0 0.15" rpy="0 0 0"/>
+      <material name="gray">
+        <color rgba="0.6 0.6 0.6 1.0"/>
+      </material>
+    </visual>
+  </link>
+  <joint name="lidar_joint" type="fixed">
+    <parent link="base_link"/>
+    <child link="lidar_link"/>
+    <origin xyz="0.11 0 0.15"/>
+  </joint>
+  <link name="camera_link">
+    <origin xyz="0.15 0 0.12" rpy="0 0 0"/>
+  </link>
+  <joint name="camera_joint" type="fixed">
+    <parent link="base_link"/>
+    <child link="camera_link"/>
+    <origin xyz="0.15 0 0.12"/>
+  </joint>
+  <xacro:macro name="wheel" params="name x y">
+    <link name="${name}_link">
       <visual>
+        <origin rpy="1.5708 0 0"/>
         <geometry>
-          <box size="${base_length} ${base_width} ${base_height}"/>
+          <cylinder radius="${wheel_radius}" length="${wheel_width}"/>
         </geometry>
-        <origin xyz="0 0 ${base_height/2}" rpy="0 0 0"/>
-        <material name="body_color">
-          <color rgba="0.15 0.15 0.18 1"/>
+        <material name="black">
+          <color rgba="0.05 0.05 0.05 1"/>
         </material>
       </visual>
       <collision>
+        <origin rpy="1.5708 0 0"/>
         <geometry>
-          <box size="${base_length} ${base_width} ${base_height}"/>
+          <cylinder radius="${wheel_radius}" length="${wheel_width}"/>
         </geometry>
-        <origin xyz="0 0 ${base_height/2}" rpy="0 0 0"/>
       </collision>
       <inertial>
-        <mass value="10.0"/>
-        <origin xyz="0 0 ${base_height/2}"/>
-        <inertia ixx="0.2" iyy="0.2" izz="0.2" ixy="0" ixz="0" iyz="0"/>
+        <mass value="1.0"/>
+        <origin xyz="0 0 0"/>
+        <inertia
+          ixx="0.01"
+          iyy="0.01"
+          izz="0.005"
+          ixy="0" ixz="0" iyz="0"/>
       </inertial>
     </link>
-    <gazebo reference="base_link">
-      <self_collide>false</self_collide>
-    </gazebo>
-    <link name="imu_link">
-      <visual>
-        <geometry>
-          <box size="0.03 0.03 0.02"/>
-        </geometry>
-        <origin xyz="0 0 0"/>
-        <material name="orange">
-          <color rgba="1 0.5 0 1"/>
-        </material>
-      </visual>
-    </link>
-    <joint name="imu_joint" type="fixed">
+    <joint name="${name}_joint" type="continuous">
       <parent link="base_link"/>
-      <child link="imu_link"/>
-      <origin xyz="0 0 0.15"/>
+      <child link="${name}_link"/>
+      <origin xyz="${x} ${y} ${wheel_radius}"/>
+      <axis xyz="0 1 0"/>
     </joint>
-    <link name="gps_link">
-      <visual>
-        <geometry>
-          <box size="0.03 0.03 0.02"/>
-        </geometry>
-        <origin xyz="0 0 0"/>
-        <material name="white">
-          <color rgba="1 1 1 1"/>
-        </material>
-      </visual>
-    </link>
-    <joint name="gps_joint" type="fixed">
-      <parent link="base_link"/>
-      <child link="gps_link"/>
-      <origin xyz="0 0 0.2"/>
-    </joint>
-    <link name="lidar_link">
-      <visual>
-        <geometry>
-          <cylinder radius="0.04" length="0.05"/>
-        </geometry>
-        <origin xyz="0 0 0"/>
-        <material name="gray">
-          <color rgba="0.6 0.6 0.6 1.0"/>
-        </material>
-      </visual>
-      <collision>
-        <geometry>
-          <cylinder radius="0.04" length="0.05"/>
-        </geometry>
-        <origin xyz="0 0 0"/>
-      </collision>
-    </link>
-    <joint name="lidar_joint" type="fixed">
-      <parent link="base_link"/>
-      <child link="lidar_link"/>
-      <origin xyz="0.11 0 0.22"/>
-    </joint>
-    <link name="camera_link"/>
-    <joint name="camera_joint" type="fixed">
-      <parent link="base_link"/>
-      <child link="camera_link"/>
-      <origin xyz="0.15 0 0.12"/>
-    </joint>
-    <xacro:macro name="wheel" params="name x y">
-      <link name="${name}_link">
-        <visual>
-          <origin rpy="1.5708 0 0"/>
-          <geometry>
-            <cylinder radius="${wheel_radius}" length="${wheel_width}"/>
-          </geometry>
-          <material name="black">
-            <color rgba="0.05 0.05 0.05 1"/>
-          </material>
-        </visual>
-        <collision>
-          <origin rpy="1.5708 0 0"/>
-          <geometry>
-            <cylinder radius="${wheel_radius}" length="${wheel_width}"/>
-          </geometry>
-        </collision>
-        <inertial>
-          <mass value="1.0"/>
-          <origin xyz="0 0 0"/>
-          <inertia ixx="0.01" iyy="0.01" izz="0.005" ixy="0" ixz="0" iyz="0"/>
-        </inertial>
-      </link>
-      <joint name="${name}_joint" type="continuous">
-        <parent link="base_link"/>
-        <child link="${name}_link"/>
-        <origin xyz="${x} ${y} ${wheel_radius}"/>
-        <axis xyz="0 1 0"/>
-      </joint>
-    </xacro:macro>
-    <xacro:wheel name="front_left_wheel"
-                 x="${wheel_x_offset}"
-                 y="${wheel_y_offset}"/>
-    <xacro:wheel name="rear_left_wheel"
-                 x="-${wheel_x_offset}"
-                 y="${wheel_y_offset}"/>
-    <xacro:wheel name="front_right_wheel"
-                 x="${wheel_x_offset}"
-                 y="-${wheel_y_offset}"/>
-    <xacro:wheel name="rear_right_wheel"
-                 x="-${wheel_x_offset}"
-                 y="-${wheel_y_offset}"/>
   </xacro:macro>
+  <xacro:wheel name="front_left_wheel"
+               x="${wheel_x_offset}"
+               y="${wheel_y_offset}"/>
+  <xacro:wheel name="rear_left_wheel"
+               x="-${wheel_x_offset}"
+               y="${wheel_y_offset}"/>
+  <xacro:wheel name="front_right_wheel"
+               x="${wheel_x_offset}"
+               y="-${wheel_y_offset}"/>
+  <xacro:wheel name="rear_right_wheel"
+               x="-${wheel_x_offset}"
+               y="-${wheel_y_offset}"/>
+</xacro:macro>
 </robot>

File: src/description/urdf/robot_sensors.xacro (robot description, xacro)
@@ -22,5 +22,5 @@
         <topic>/scan</topic>
         <visualize>true</visualize>
-        <gz_frame_id>lidar_link</gz_frame_id>
+        <frame_id>lidar_link</frame_id>
         <lidar>
           <scan>
