Commit message: Revert "merge (#30)"
This reverts commit f7f2a340510130d97a0e781ddb53dca27cd18fd7.

File: src/description/urdf/robot.urdf.xacro (robot description, xacro)
@@ -1,12 +1,49 @@
 <?xml version="1.0"?>
-<robot name="skid_steer_bot"
-       xmlns:xacro="http://www.ros.org/wiki/xacro">
-  <xacro:include filename="robot_base.xacro"/>
-  <xacro:include filename="robot_control.xacro"/>
-  <xacro:include filename="robot_sim.xacro"/>
-  <xacro:include filename="robot_sensors.xacro"/>
-  <xacro:base/>
-  <xacro:control/>
-  <xacro:sim/>
-  <xacro:sensors/>
+<robot name="mercury" xmlns:xacro="http://www.ros.org/wiki/xacro">
+  <!-- ================= BASE ================= -->
+  <link name="base_link">
+    <visual>
+      <geometry>
+        <box size="0.4 0.3 0.1"/>
+      </geometry>
+      <origin xyz="0 0 0.05"/>
+    </visual>
+  </link>
+  <!-- ================= LIDAR ================= -->
+  <link name="laser_link">
+    <visual>
+      <geometry>
+        <cylinder length="0.05" radius="0.05"/>
+      </geometry>
+    </visual>
+  </link>
+  <joint name="laser_joint" type="fixed">
+    <parent link="base_link"/>
+    <child link="laser_link"/>
+    <origin xyz="0.2 0 0.15" rpy="0 0 0"/>
+  </joint>
+  <!-- ================= REALSENSE CAMERA BODY ================= -->
+  <link name="camera_link"/>
+  <joint name="camera_mount_joint" type="fixed">
+    <parent link="base_link"/>
+    <child link="camera_link"/>
+    <!-- Adjust these values to your real mounting -->
+    <origin xyz="0.15 0 0.12" rpy="0 0 0"/>
+  </joint>
+  <!-- ================= IMU FRAME ================= -->
+  <link name="camera_imu_frame"/>
+  <joint name="camera_imu_joint" type="fixed">
+    <parent link="camera_link"/>
+    <child link="camera_imu_frame"/>
+    <origin xyz="0 0 0" rpy="0 0 0"/>
+  </joint>
+  <!-- ================= IMU OPTICAL FRAME ================= -->
+  <!-- Optical frame rotation: X right, Y down, Z forward -->
+  <link name="camera_imu_optical_frame"/>
+  <joint name="camera_imu_optical_joint" type="fixed">
+    <parent link="camera_imu_frame"/>
+    <child link="camera_imu_optical_frame"/>
+    <!-- Convert from ROS frame to optical frame -->
+    <origin xyz="0 0 0" rpy="-1.5708 0 -1.5708"/>
+  </joint>
 </robot>
